Commit message: ok to run moveit but have self-collision

File: isaac_manipulator_pick_and_place/urdf/ur10e_robotiq_hande.urdf (robot description, URDF)
Before this commit: robot ur10e_robot, 18 links, 17 joints
Joints:
- joint gripper_joint: parent robotiq_base_link -> robotiq_hande_coupler
- joint robotiq_hande_coupler_joint: origin xyz=0 0 0.00695 rpy=0 0 ${-pi/2.0} -> xyz=0 0 0.00695 rpy=0 0 -1.57

File: isaac_manipulator_pick_and_place/urdf/ur_robotiq_hande.urdf.xacro (robot description, xacro)
@@ -27,5 +27,6 @@
         parent="tool0"
         tty="$(arg com_port)"
-        use_fake_hardware="$(arg use_fake_hardware)"/>
+        use_fake_hardware="true"/>
+        <!-- use_fake_hardware="$(arg use_fake_hardware)"/> -->
     <link name="gripper_frame">
         <inertial>

Commit message: Write most of the README in terms of running with self-defined objects

File: isaac_manipulator_pick_and_place/urdf/ur10e_robotiq_hande.urdf (robot description, URDF)
Before this commit: robot ur10e_robot, 18 links, 17 joints
Links:
- link base_link_inertia: geometry collision mesh filename=package://isaac_manipulator_pick_and_place/meshes/ur10e/col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; visual mesh filename=meshes/ur10e/visual/base.dae
- link forearm_link: geometry collision mesh filename=package://isaac_manipulator_pick_and_place/meshes/ur10e/col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; visual mesh filename=package://isaac_manipulator_pick_and_place/meshes/ur10e/vis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
- link robotiq_hande_coupler: geometry collision cylinder length=0.0139 radius=0.0375; visual mesh filename=package://isaac_manipulator_pick_and_place/meshes/robotiq_h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
- link robotiq_hande_left_finger: geometry collision mesh filename=package://isaac_manipulator_pick_and_place/meshes/robotiq_h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 scale=1.0 1.0 1.0; visual mesh filename=package://isaac_manipulator_pick_and_place/meshes/robotiq_h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 scale=1.0 1.0 1.0
- link robotiq_hande_link: geometry collision cylinder length=0.0988 radius=0.0375; visual mesh filename=package://isaac_manipulator_pick_and_place/meshes/robotiq_h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 scale=1.0 1.0 1.0
- link robotiq_hande_right_finger: geometry collision mesh filename=package://isaac_manipulator_pick_and_place/meshes/robotiq_h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 scale=1.0 1.0 1.0; visual mesh filename=package://isaac_manipulator_pick_and_place/meshes/robotiq_h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 scale=1.0 1.0 1.0
- link shoulder_link: geometry collision mesh filename=package://isaac_manipulator_pick_and_place/meshes/ur10e/col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; visual mesh filename=package://isaac_manipulator_pick_and_place/meshes/ur10e/vis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
- link upper_arm_link: geometry collision mesh filename=package://isaac_manipulator_pick_and_place/meshes/ur10e/col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; visual mesh filename=package://isaac_manipulator_pick_and_place/meshes/ur10e/vis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
- link wrist_1_link: geometry collision mesh filename=package://isaac_manipulator_pick_and_place/meshes/ur10e/col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; visual mesh filename=package://isaac_manipulator_pick_and_place/meshes/ur10e/vis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
- link wrist_2_link: geometry collision mesh filename=package://isaac_manipulator_pick_and_place/meshes/ur10e/col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; visual mesh filename=package://isaac_manipulator_pick_and_place/meshes/ur10e/vis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
- link wrist_3_link: geometry collision mesh filename=package://isaac_manipulator_pick_and_place/meshes/ur10e/col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; visual mesh filename=package://isaac_manipulator_pick_and_place/meshes/ur10e/vis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

Commit message: Fix Joint Limit problem.

File: isaac_manipulator_pick_and_place/urdf/ur10e_robotiq_hande.urdf (robot description, URDF)
Before this commit: robot ur10e_robot, 18 links, 17 joints
Joints:
- joint shoulder_pan_joint: limit lower=-6.283185307179586 upper=6.283185307179586 effort=330.0 velocity=2.0943951023931953 -> lower=-3.141592653589793 upper=0.0 effort=330.0 velocity=2.0943951023931953
